File: hardware/control_board/connector.kicad_sch (KiCad schematic)
At the start: 0 parts

Commit message: added connectors
Parts:
- added J3, J4: TX24-60R-6ST-H1E, Library:JAE_TX24-60R-6ST-H1E, symbol Library:TX24-60R-6ST-H1E
